File: ai03-pcb-guide.kicad_pcb (KiCad board)
At the start: 2 copper layers, 24 parts, among them SW1 SW_Push, U1 ATmega32U4-AU, Y1 Crystal_GND24_Small

Commit message: Completes pcb creation
Routing:
- added copper zone on B.Cu, net GND
Other:
- board text added: "Hello World!"
Changed lines of the file:
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@@
   (general
     (thickness 1.6)
-    (drawings 11)
+    (drawings 12)
     (tracks 236)
     (zones 0)
@@
       (rotate (xyz 0 0 0))
     )
+  )
+  (gr_text "Hello World!" (at 122.0343 64.8843) (layer F.SilkS)
+    (effects (font (size 1 1) (thickness 0.15)))
   )
   (gr_line (start 42.8625 101.6) (end 47.625 101.6) (layer F.SilkS) (width 0.12))
@@
   (segment (start 144.4903 71.4385) (end 144.6403 71.4385) (width 0.254) (layer B.Cu) (net 6))
   (segment (start 141.6403 68.5885) (end 144.4903 71.4385) (width 0.254) (layer B.Cu) (net 6))
-  (segment (start 139.2028 68.5885) (end 141.6403 68.5885) (width 0.254) (layer B.Cu) (net 6))
+  (segment (start 141.6403 68.5885) (end 139.2028 68.5885) (width 0.254) (layer B.Cu) (net 6))
   (segment (start 145.4943 74.7385) (end 145.4953 74.7395) (width 0.254) (layer B.Cu) (net 7))
   (segment (start 144.6403 74.7385) (end 145.4943 74.7385) (width 0.254) (layer B.Cu) (net 7))
@@
   (segment (start 91.275 85.725) (end 90.069 86.931) (width 0.254) (layer B.Cu) (net 20))
   (segment (start 92.075 85.725) (end 91.275 85.725) (width 0.254) (layer B.Cu) (net 20))
+  (zone (net 1) (net_name GND) (layer B.Cu) (hatch edge 0.508)
+    (connect_pads (clearance 0.508))
+    (min_thickness 0.254)
+    (fill yes (arc_segments 32) (thermal_gap 0.508) (thermal_bridge_width 0.508))
+    (polygon
+      (pts
+        (xy 37.592 62.0522) (xy 37.4904 104.4448) (xy 127.1905 103.4034) (xy 127.127 61.4172)
+      )
+    )
+  )
+  (zone (net 1) (net_name GND) (layer B.Cu) (hatch edge 0.508)
+    (connect_pads (clearance 0.508))
+    (min_thickness 0.254)
+    (fill yes (arc_segments 32) (thermal_gap 0.508) (thermal_bridge_width 0.508))
+    (polygon
+      (pts
+        (xy 94.9579 81.2165) (xy 94.6658 98.0313) (xy 127.3937 98.9838) (xy 127.0254 80.0481) (xy 126.9492 80.1624)
+      )
+    )
+  )
 )
